Commit message: added node parameters for arm_controller_node

File: arm_description/urdf/arm.urdf.xacro (robot description, xacro)
@@ -379,8 +379,8 @@
     </hardware>
     <!-- Hardware Interface macro call -->
-    <xacro:arm_hardware_interface joint_name="j0" initial_pos="0.0"/>
-    <xacro:arm_hardware_interface joint_name="j1" initial_pos="0.0"/>
-    <xacro:arm_hardware_interface joint_name="j2" initial_pos="0.0"/>
-    <xacro:arm_hardware_interface joint_name="j3" initial_pos="0.0"/>
+    <xacro:position_joint_interface joint_name="j0" initial_pos="0.0"/>
+    <xacro:position_joint_interface joint_name="j1" initial_pos="0.0"/>
+    <xacro:position_joint_interface joint_name="j2" initial_pos="0.0"/>
+    <xacro:position_joint_interface joint_name="j3" initial_pos="0.0"/>
   </ros2_control>
   <!-- Sensors macro include -->

File: arm_description/urdf/arm_hardware_interface.xacro (robot description, xacro)
@@ -1,5 +1,5 @@
 <?xml version="1.0"?>
 <robot xmlns:xacro="http://ros.org/wiki/xacro">
-    <xacro:macro name="arm_hardware_interface" params="joint_name initial_pos">
+    <xacro:macro name="position_joint_interface" params="joint_name initial_pos">
         <joint name="${joint_name}">
             <!-- Command Interface -->

Commit message: modified color in urdf and xacro

File: arm_description/urdf/arm.urdf.xacro (robot description, xacro)
@@ -3,4 +3,8 @@
   <material name="red">
     <color rgba="1 0 0 1"/>
+  </material>
+  <!-- Material Black for Dynamixel motor -->
+  <material name="black">
+      <color rgba="0 0 0 1"/>
   </material>
   <link name="base_link">
@@ -83,4 +87,5 @@
       </geometry>
       <origin rpy="0 0 0" xyz="0 0 0"/>
+      <material name="black"/>
     </visual>
     <collision>
@@ -139,4 +144,5 @@
       </geometry>
       <origin rpy="0 0 0" xyz="0 0 0"/>
+      <material name="black"/>
     </visual>
     <collision>
@@ -194,4 +200,5 @@
       </geometry>
       <origin rpy="0 0 0" xyz="0 0 0"/>
+      <material name="black"/>
     </visual>
     <collision>
@@ -250,4 +257,5 @@
       </geometry>
       <origin rpy="0 0 0" xyz="0 0 0"/>
+      <material name="black"/>
     </visual>
     <collision>

Commit message: added world frame

File: arm_description/urdf/arm.urdf.xacro (robot description, xacro)
@@ -8,4 +8,11 @@
       <color rgba="0 0 0 1"/>
   </material>
+  <!-- Add world reference -->
+  <link name="world"/>
+  <joint name="base_joint" type="fixed">
+    <origin rpy="0.0 0 0" xyz="0 0 0"/>
+    <parent link="world"/>
+    <child link="base_link"/>
+  </joint>
   <link name="base_link">
     <visual>

Commit message: bug fix

File: arm_description/urdf/arm.urdf.xacro (robot description, xacro)
@@ -8,11 +8,4 @@
       <color rgba="0 0 0 1"/>
   </material>
-  <!-- Add world reference -->
-  <link name="world"/>
-  <joint name="base_joint" type="fixed">
-    <origin rpy="0.0 0 0" xyz="0 0 0"/>
-    <parent link="world"/>
-    <child link="base_link"/>
-  </joint>
   <link name="base_link">
     <visual>
@@ -363,8 +356,9 @@
   </link>
   <!-- camera link and camera joint -->
+  <!--origin xyz="0.5 -0.3 0.6" rpy="0.0 0.5 -3.66"/-->
   <joint name="camera_joint" type="fixed">
     <parent link="base_link"/>
     <child link="camera_link"/>
-    <origin xyz="0.5 -0.3 0.6" rpy="0.0 0.5 -3.66"/>
+    <origin xyz="0 0 0" rpy="0 0 -1.57"/>
   </joint>
   <material name="grey">

File: arm_description/urdf/arm_camera.xacro (robot description, xacro)
@@ -1,23 +1,24 @@
 <?xml version="1.0"?>
 <robot xmlns:xacro="http://www.ros.org/wiki/xacro">
+    <!-- Camera sensor porperties -->
     <xacro:macro name="arm_camera">
         <gazebo reference="camera_link">
-        <sensor name="camera" type="camera">
-            <camera>
-            <horizontal_fov>1.047</horizontal_fov>
-            <image>
-                <width>320</width>
-                <height>240</height>
-            </image>
-            <clip>
-                <near>0.1</near>
-                <far>100</far>
-            </clip>
-            </camera>
-            <always_on>1</always_on>
-            <update_rate>30</update_rate>
-            <visualize>true</visualize>
-            <topic>camera</topic>
-        </sensor>
+            <sensor name="camera" type="camera">
+                <camera>
+                <horizontal_fov>1.047</horizontal_fov>
+                <image>
+                    <width>320</width>
+                    <height>240</height>
+                </image>
+                <clip>
+                    <near>0.1</near>
+                    <far>100</far>
+                </clip>
+                </camera>
+                <always_on>1</always_on>
+                <update_rate>30</update_rate>
+                <visualize>true</visualize>
+                <topic>camera</topic>
+            </sensor>
         </gazebo>
     </xacro:macro>

File: arm_description/urdf/arm_hardware_interface.xacro (robot description, xacro)
@@ -1,9 +1,11 @@
 <?xml version="1.0"?>
+<!-- macro for creating a joint with a command and feedback interfaces -->
 <robot xmlns:xacro="http://ros.org/wiki/xacro">
     <xacro:macro name="position_joint_interface" params="joint_name initial_pos">
+     <!-- Define a joint element -->
         <joint name="${joint_name}">
             <!-- Command Interface -->
             <command_interface name="position"/>
-            <!-- Feedback state Interface -->
+            <!-- Feedback state Interface (position, velocity, effort)-->
             <state_interface name="position">
                 <param name="initial_value">${initial_pos}</param>
